File: hardware/pcb/welld.kicad_sch (KiCad schematic)
At the start: 70 parts, among them J1 LiPo, J10 PROG_6pin, J12 SolarPanel, J2 USB-C, J3 U.FL_Antenna, J4 4-20mA_CH1, J5 4-20mA_CH2, J6 DS18B20, J7 Spare, J8 I2C_4pin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

Commit message: Bring PCB schematic/layout in sync with the design docs
The KiCad generator was a revision behind the design notes and BOM:
the 12 V boost (U8), external ADC (U9), fuel gauge (U10), charger
interlock (Q1/Q2), boost inductor (L1), solar TVS (D8) and their
passives were documented but absent from welld.kicad_sch/.kicad_pcb.
Add them to generate_kicad.py, with TPS61023/ADS1115/MAX17048 symbols,
and regenerate.

Fix schematic/layout bugs: duplicate ESP32-C6 pin number, missing
GPIO14, stale DW01A symbol (now S-8261A), JST PH footprint on J1
(now JST XH), ADS1115 SOIC-8 footprint (now MSOP-10/VSSOP-10, the
correct 10-pin package), and two off-board component placements.
Add the missing TP4056 CE pull-up (R29).

Correct design.md errors: the R23/R24 boost-divider values, the D8
TVS protection claim, the reverse-polarity FET topology, the ESP32-C6
USB pin assignment, the ADS1115 channel/PGA description, and add a
GPIO15 strapping note and an MPPT diode-drop note.

Drop all revision language across the hardware docs and generators —
this is the single current design.

https://claude.ai/code/session_01QqBrArSSEuu1qysbVH7Nqt
Parts:
- removed U3: DW01A, symbol welld:DW01A
- added C19, C22: 10uF, symbol Device:C
- added C20: 22uF, symbol Device:C
- added C21: 100nF, symbol Device:C
- added D7: LED DNF, symbol Device:LED
- added D8: SMAJ7.0A, symbol Device:D_TVS
- added L1: 4.7uH, symbol Device:L
- added Q1, Q2: BSS123, symbol Device:Q_NMOS_GSD
- added R23: 1.1M, symbol Device:R
- added R24: 47k, symbol Device:R
- added R25, R26, R27, R29: 4.7k, symbol Device:R
- added R28: 100R, symbol Device:R
- added SJ1: VBOOST_EN DNF, symbol Jumper:SolderJumper_2_Open
- added SJ2: VLOOP_BUS, symbol Jumper:SolderJumper_2_Open
- added SJ3: LED_DIS, symbol Jumper:SolderJumper_2_Open
- added SJ4: UART_TX DNF, symbol Jumper:SolderJumper_2_Open
- added SJ5: UART_RX DNF, symbol Jumper:SolderJumper_2_Open
- added U10: MAX17048, symbol welld:MAX17048
- added U3: S-8261AAYFT, symbol welld:S8261A
- added U8: TPS61023, symbol welld:TPS61023
- added U9: ADS1115, symbol welld:ADS1115
