File: hardware/pcb/welld.kicad_sch (KiCad schematic)
At the start: 94 parts, among them J1 LiPo, J10 PROG_6pin, J12 SolarPanel, J2 USB-C, J3 U.FL_Antenna, J4 4-20mA_CH1, J5 4-20mA_CH2, J6 DS18B20, J7 Spare, J8 I2C_4pin, J9 GPIO_8pin, Q1 BSS123, Q2 BSS123, SW1 RESET, SW2 BOOT, U1 TPS7A0533, U10 MAX17048, U2 TP4056, U3 S-8261AAYFT, U4 FS8205A, U5 USBLC6-2SC6, U6 ESP32-C6-MINI, U7 CN3791, U8 TPS61023, U9 ADS1115

Commit message: PCB analog/protection/interlock fixes + three new agents
Analog front-end:
- C3, C5: 100nF → 1µF to lower RC filter corner from 15.9kHz to 1.6kHz
- Add FB1 (BLM18KG601SN1D ferrite) + C23/C24 (ADS1115 VDD bypass) to isolate
  the 16-bit ADC supply from TPS61023 switching noise and 2.4GHz radio

Transient protection:
- Add D9/D10 (SMAJ5.0CA, bidirectional, 400W) at J4/J5 SIG terminals before
  the shunt resistors — IEC 61000-4-5 surge protection for well-head cables
- Add D11 (SMAJ13A, 13V standoff, 400W) on VLOOP rail between U8 and field
  terminals to clamp cable back-EMF and lightning-induced transients

Charger interlock:
- Fix GPIO6 polarity throughout: CN3791 CHRG is active-LOW (was documented
  as active-high in CLAUDE.md and design.md GPIO table)
- Fix design.md: CN3791 has no EN/shutdown pin; GPIO6 reads CHRG output only
- Add Q3 (BSS84 P-ch) hardware interlock: gate=/CHRG_SOLAR, source=CE node,
  drain=GND; eliminates the boot-window race without firmware involvement
- Add R30 (10kΩ) as Q3 gate pull-up to +3V3

Agents:
- Add test-engineer, docs-writer, ci-engineer agents to .claude/agents/
- Expand CLAUDE.md Sub-Agent Routing Rules with full responsibility table
  and handoff order for hardware vs firmware-only changes

Co-Authored-By: Claude Sonnet 4.6 <noreply@anthropic.com>
Parts:
- added C23: 100nF, symbol Device:C
- added C24: 1uF, symbol Device:C
- added D10, D9: SMAJ5.0CA, symbol Device:D_TVS_Bidirectional
- added D11: SMAJ13A, symbol Device:D_TVS
- added FB1: BLM18KG601SN1D, symbol Device:L
- added Q3: BSS84, symbol Device:Q_PMOS_GSD
- added R30: 10k, symbol Device:R
- C3, C5: value 100nF -> 1uF
Changed lines of the file:
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@@
   (title_block
     (title "WellD Well-Level Monitor")
-    (date "2026-05-16")
+    (date "2026-05-18")
     (company "WellD Project")
     (comment 1 "ESP32-C6-MINI-1U + TP4056 + CN3791 + TPS7A0533 + TPS61023")
@@
   )
   (global_label "MAX_ALRT" (shape input) (at 340.00 360.00 0) (fields_autoplaced)
+    (effects (font (size 1.27 1.27)) (justify left))
+    (property "Intersheets" "" (at 0 0 0) (effects (font (size 1.27 1.27)) (hide yes)))
+  )
+  (global_label "LOOP_TERM_CH1" (shape passive) (at 415.00 175.00 0) (fields_autoplaced)
+    (effects (font (size 1.27 1.27)) (justify left))
+    (property "Intersheets" "" (at 0 0 0) (effects (font (size 1.27 1.27)) (hide yes)))
+  )
+  (global_label "LOOP_TERM_CH2" (shape passive) (at 445.00 175.00 0) (fields_autoplaced)
+    (effects (font (size 1.27 1.27)) (justify left))
+    (property "Intersheets" "" (at 0 0 0) (effects (font (size 1.27 1.27)) (hide yes)))
+  )
+  (global_label "+3V3_ADS" (shape passive) (at 60.00 280.00 0) (fields_autoplaced)
     (effects (font (size 1.27 1.27)) (justify left))
     (property "Intersheets" "" (at 0 0 0) (effects (font (size 1.27 1.27)) (hide yes)))
@@
       (effects (font (size 1.27 1.27)) (hide yes)))
   )
+  (symbol (lib_id "Device:D_TVS_Bidirectional") (at 420.00 185.00 0) (unit 1)
+    (in_bom yes) (on_board yes) (dnp no) (fields_autoplaced)
+    (property "Reference" "D9" (at 420.00 181.19 0)
+      (effects (font (size 1.27 1.27))))
+    (property "Value" "SMAJ5.0CA" (at 420.00 188.81 0)
+      (effects (font (size 1.27 1.27))))
+    (property "Footprint" "" (at 0 0 0)
+      (effects (font (size 1.27 1.27)) (hide yes)))
+    (property "Datasheet" "~" (at 0 0 0)
+      (effects (font (size 1.27 1.27)) (hide yes)))
+  )
   (symbol (lib_id "Device:C") (at 460.00 225.00 0) (unit 1)
     (in_bom yes) (on_board yes) (dnp no) (fields_autoplaced)
     (property "Reference" "C3" (at 460.00 221.19 0)
       (effects (font (size 1.27 1.27))))
-    (property "Value" "100nF" (at 460.00 228.81 0)
+    (property "Value" "1uF" (at 460.00 228.81 0)
       (effects (font (size 1.27 1.27))))
     (property "Footprint" "" (at 0 0 0)
@@
       (effects (font (size 1.27 1.27)) (hide yes)))
   )
+  (symbol (lib_id "Device:D_TVS_Bidirectional") (at 450.00 185.00 0) (unit 1)
+    (in_bom yes) (on_board yes) (dnp no) (fields_autoplaced)
+    (property "Reference" "D10" (at 450.00 181.19 0)
+      (effects (font (size 1.27 1.27))))
+    (property "Value" "SMAJ5.0CA" (at 450.00 188.81 0)
+      (effects (font (size 1.27 1.27))))
+    (property "Footprint" "" (at 0 0 0)
+      (effects (font (size 1.27 1.27)) (hide yes)))
+    (property "Datasheet" "~" (at 0 0 0)
+      (effects (font (size 1.27 1.27)) (hide yes)))
+  )
   (symbol (lib_id "Device:C") (at 500.00 225.00 0) (unit 1)
     (in_bom yes) (on_board yes) (dnp no) (fields_autoplaced)
     (property "Reference" "C5" (at 500.00 221.19 0)
       (effects (font (size 1.27 1.27))))
-    (property "Value" "100nF" (at 500.00 228.81 0)
+    (property "Value" "1uF" (at 500.00 228.81 0)
       (effects (font (size 1.27 1.27))))
     (property "Footprint" "" (at 0 0 0)
@@
       (effects (font (size 1.27 1.27)) (hide yes)))
   )
+  (symbol (lib_id "Device:L") (at 60.00 285.00 0) (unit 1)
+    (in_bom yes) (on_board yes) (dnp no) (fields_autoplaced)
+    (property "Reference" "FB1" (at 60.00 281.19 0)
+      (effects (font (size 1.27 1.27))))
+    (property "Value" "BLM18KG601SN1D" (at 60.00 288.81 0)
+      (effects (font (size 1.27 1.27))))
+    (property "Footprint" "" (at 0 0 0)
+      (effects (font (size 1.27 1.27)) (hide yes)))
+    (property "Datasheet" "~" (at 0 0 0)
+      (effects (font (size 1.27 1.27)) (hide yes)))
+  )
+  (symbol (lib_id "Device:C") (at 80.00 285.00 0) (unit 1)
+    (in_bom yes) (on_board yes) (dnp no) (fields_autoplaced)
+    (property "Reference" "C23" (at 80.00 281.19 0)
+      (effects (font (size 1.27 1.27))))
+    (property "Value" "100nF" (at 80.00 288.81 0)
+      (effects (font (size 1.27 1.27))))
+    (property "Footprint" "" (at 0 0 0)
+      (effects (font (size 1.27 1.27)) (hide yes)))
+    (property "Datasheet" "~" (at 0 0 0)
+      (effects (font (size 1.27 1.27)) (hide yes)))
+  )
+  (symbol (lib_id "Device:C") (at 90.00 285.00 0) (unit 1)
+    (in_bom yes) (on_board yes) (dnp no) (fields_autoplaced)
+    (property "Reference" "C24" (at 90.00 281.19 0)
+      (effects (font (size 1.27 1.27))))
+    (property "Value" "1uF" (at 90.00 288.81 0)
+      (effects (font (size 1.27 1.27))))
+    (property "Footprint" "" (at 0 0 0)
+      (effects (font (size 1.27 1.27)) (hide yes)))
+    (property "Datasheet" "~" (at 0 0 0)
+      (effects (font (size 1.27 1.27)) (hide yes)))
+  )
   (symbol (lib_id "welld:ADS1115") (at 80.00 300.00 0) (unit 1)
     (in_bom yes) (on_board yes) (dnp no) (fields_autoplaced)
@@
       (effects (font (size 1.27 1.27)) (hide yes)))
   )
+  (symbol (lib_id "Device:Q_PMOS_GSD") (at 160.00 315.00 0) (unit 1)
+    (in_bom yes) (on_board yes) (dnp no) (fields_autoplaced)
+    (property "Reference" "Q3" (at 160.00 311.19 0)
+      (effects (font (size 1.27 1.27))))
+    (property "Value" "BSS84" (at 160.00 318.81 0)
+      (effects (font (size 1.27 1.27))))
+    (property "Footprint" "" (at 0 0 0)
+      (effects (font (size 1.27 1.27)) (hide yes)))
+    (property "Datasheet" "~" (at 0 0 0)
+      (effects (font (size 1.27 1.27)) (hide yes)))
+  )
   (symbol (lib_id "Device:R") (at 200.00 315.00 0) (unit 1)
     (in_bom yes) (on_board yes) (dnp no) (fields_autoplaced)
@@
       (effects (font (size 1.27 1.27)) (hide yes)))
   )
+  (symbol (lib_id "Device:R") (at 160.00 330.00 0) (unit 1)
+    (in_bom yes) (on_board yes) (dnp no) (fields_autoplaced)
+    (property "Reference" "R30" (at 160.00 326.19 0)
+      (effects (font (size 1.27 1.27))))
+    (property "Value" "10k" (at 160.00 333.81 0)
+      (effects (font (size 1.27 1.27))))
+    (property "Footprint" "" (at 0 0 0)
+      (effects (font (size 1.27 1.27)) (hide yes)))
+    (property "Datasheet" "~" (at 0 0 0)
+      (effects (font (size 1.27 1.27)) (hide yes)))
+  )
   (symbol (lib_id "Device:LED") (at 40.00 315.00 0) (unit 1)
     (in_bom yes) (on_board yes) (dnp no) (fields_autoplaced)
@@
       (effects (font (size 1.27 1.27))))
     (property "Footprint" "" (at 0 0 0)
+      (effects (font (size 1.27 1.27)) (hide yes)))
+    (property "Datasheet" "~" (at 0 0 0)
+      (effects (font (size 1.27 1.27)) (hide yes)))
+  )
+  (symbol (lib_id "Device:D_TVS") (at 260.00 300.00 0) (unit 1)
+    (in_bom yes) (on_board yes) (dnp no) (fields_autoplaced)
+    (property "Reference" "D11" (at 260.00 296.19 0)
+      (effects (font (size 1.27 1.27))))
+    (property "Value" "SMAJ13A" (at 260.00 303.81 0)
+      (effects (font (size 1.27 1.27))))
+    (property "Footprint" "" (at 0 0 0)

Commit message: feat: PCB thermal/testpoints/decoupling, firmware robustness, Kconfig cleanup
PCB:
- CN3791 (U7): 10×10 mm GND thermal copper pour F.Cu+B.Cu with 4 thermal vias;
  handles 1.75 W worst-case simultaneous solar+boost load
- TPS61023 (U8): GND via-stitch ring around boost island for low-inductance return
- TP1–TP14: 1.0 mm SMD test points (DNF) for VBAT, VLOOP, 3V3, GND, LOOP+/-,
  SDA, SCL, 1WIRE, VSOLAR, VBAT_RAW, DRDY, ALRT, /CHRG
- C25, C26: 100 nF 0402 bypass caps on MAX17048 VDD and S-8261 VCC (previously missing)

Firmware:
- MAX17048 ALRT (GPIO14): startup level check + full STATUS flag decode
  (RI/VH/VL/VR/HD/SC) before clearing; replaces partial VL-only clear
- I2C bus recovery: 9-pulse SCL clock sequence on SDA-stuck detection at init
- Short-circuit detection: sensor_read_level() returns -2.0 for >21 mA loop current
- ADC oversampling (WELLD_ADC_OVERSAMPLE_ENABLED, default off): median-of-3 reads;
  opt-in for noisy installations
- Temperature compensation (WELLD_TEMP_COMPENSATION_ENABLED, default off):
  water-density correction at configurable ppm/°C
- DS18B20 resolution (WELLD_DS18B20_RESOLUTION_BITS, default 12-bit): saves up to
  656 ms/wakeup at 9-bit
- OTA rollback guard: RTC boot-attempt counter, rolls back partition after 3 fails
- Factory reset GPIO (WELLD_FACTORY_RESET_GPIO, default GPIO13): hold LOW at boot

Kconfig:
- Moved WELLD_ADC_OVERSAMPLE_ENABLED, WELLD_TEMP_COMPENSATION_*, WELLD_DS18B20_*,
  and WELLD_SOLAR_DETECT_GPIO from main/Kconfig.projbuild to components/sensor/Kconfig
  so standalone test/sensor build can see them; fixes CI on-device build failure

Co-Authored-By: Claude Sonnet 4.6 <noreply@anthropic.com>
Parts:
- added C25, C26: 100nF, symbol Device:C
- added C_SH1, C_SH2: 10nF, symbol Device:C
- added R31: 10k, symbol Device:R
- added R32: 33R DNF, symbol Device:R
- added TP1: VBAT, symbol welld:TestPoint_Pad
- added TP10: VSOLAR_IN, symbol welld:TestPoint_Pad
- added TP11: VBAT_RAW, symbol welld:TestPoint_Pad
- added TP12: ADS_DRDY, symbol welld:TestPoint_Pad
- added TP13: MAX_ALRT, symbol welld:TestPoint_Pad
- added TP14: /CHRG_SOLAR, symbol welld:TestPoint_Pad
- added TP2: VLOOP, symbol welld:TestPoint_Pad
- added TP3: +3V3, symbol welld:TestPoint_Pad
- added TP4: GND, symbol welld:TestPoint_Pad
- added TP5: LOOP_TERM_CH1, symbol welld:TestPoint_Pad
- added TP6: LOOP_TERM_CH2, symbol welld:TestPoint_Pad
- added TP7: 1WIRE, symbol welld:TestPoint_Pad
- added TP8: I2C_SDA, symbol welld:TestPoint_Pad
- added TP9: I2C_SCL, symbol welld:TestPoint_Pad
- D10, D9: value SMAJ5.0CA -> SMAJ3.3CA

Commit message: feat: 2S1P design — dual solar+USB-C charging, firmware, Z2M, PCB, case
Sinowatt 2S1P 18650 pack (6.0–8.4 V). Two independent charging paths:
- CN3722 MPPT solar charger via J12 screw terminal (GPIO6 /CHRG status)
- TP5100 USB-C boost charger via J13 connector (GPIO4 CE control)

PCB: AP63205 buck, MT3608B VLOOP boost, ADS1115 ADC, JST PH 2.0 mm battery
connector. SOC via resistor divider (BATT_DIVIDER_RATIO=430, FULL=8400 mV,
EMPTY=6000 mV). Firmware drives GPIO4 HIGH on wake to enable USB charging and
isolates it before deep-sleep so R37 passively holds CE LOW.

Case: battery bay 41×71×22 mm pocket for 2S1P pack; USB-C slot on left wall
for J13; programming gland repositioned to clear USB-C slot.

Z2M: 2S voltage thresholds and solar charge status reporting.

Tests: 2/2 host, 34/34 Z2M converter — all green.

Co-Authored-By: Claude Sonnet 4.6 <noreply@anthropic.com>
Parts:
- D8: value SMAJ7.0A -> SMAJ28CA
- J1: value LiPo -> LiPo_2S_JST-PH2
- R23: value 1.1M -> 1.9M
- R24: value 47k -> 100k
- R7: value 100k -> 330k
- TP11: value VBAT_RAW -> VBAT_RAW_2S
- TP13: value MAX_ALRT -> REMOVED_MAX_ALRT
- TP14: value /CHRG_SOLAR -> REMOVED_CHRG_SOLAR
- U1: value TPS7A0533 -> AP63205WU
- U7: value CN3791 -> CN3722
- U8: value TPS61023 -> MT3608B
Changed lines of the file:
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@@
     (date "2026-05-18")
     (company "WellD Project")
-    (comment 1 "ESP32-C6-MINI-1U + TP4056 + CN3791 + TPS7A0533 + TPS61023")
+    (comment 1 "ESP32-C6-MINI-1U + CN3722 + AP63205 + MT3608B (2S 18650 LiPo)")
   )
   (global_label "VSOLAR_IN" (shape passive) (at 30.00 15.00 0) (fields_autoplaced)
@@
     (property "Intersheets" "" (at 0 0 0) (effects (font (size 1.27 1.27)) (hide yes)))
   )
-  (global_label "VUSB_IN" (shape passive) (at 30.00 120.00 0) (fields_autoplaced)
-    (effects (font (size 1.27 1.27)) (justify left))
-    (property "Intersheets" "" (at 0 0 0) (effects (font (size 1.27 1.27)) (hide yes)))
-  )
-  (global_label "VUSB" (shape passive) (at 80.00 120.00 0) (fields_autoplaced)
-    (effects (font (size 1.27 1.27)) (justify left))
-    (property "Intersheets" "" (at 0 0 0) (effects (font (size 1.27 1.27)) (hide yes)))
-  )
+  ;; VUSB_IN and VUSB labels removed — USB-C charging path deleted in 2S redesign
   (global_label "VBAT" (shape passive) (at 210.00 70.00 0) (fields_autoplaced)
     (effects (font (size 1.27 1.27)) (justify left))
@@
     (property "Intersheets" "" (at 0 0 0) (effects (font (size 1.27 1.27)) (hide yes)))
   )
-  (global_label "/CHRG_USB" (shape passive) (at 180.00 120.00 0) (fields_autoplaced)
-    (effects (font (size 1.27 1.27)) (justify left))
-    (property "Intersheets" "" (at 0 0 0) (effects (font (size 1.27 1.27)) (hide yes)))
-  )
-  (global_label "/DONE_USB" (shape passive) (at 180.00 130.00 0) (fields_autoplaced)
-    (effects (font (size 1.27 1.27)) (justify left))
-    (property "Intersheets" "" (at 0 0 0) (effects (font (size 1.27 1.27)) (hide yes)))
-  )
+  ;; /CHRG_USB and /DONE_USB labels removed — TP4056 deleted in 2S redesign
   (global_label "/CHRG_SOLAR" (shape passive) (at 120.00 45.00 0) (fields_autoplaced)
     (effects (font (size 1.27 1.27)) (justify left))
@@
     (property "Intersheets" "" (at 0 0 0) (effects (font (size 1.27 1.27)) (hide yes)))
   )
-  (global_label "CHRG_USB_DIS" (shape input) (at 180.00 360.00 0) (fields_autoplaced)
-    (effects (font (size 1.27 1.27)) (justify left))
-    (property "Intersheets" "" (at 0 0 0) (effects (font (size 1.27 1.27)) (hide yes)))
-  )
+  ;; CHRG_USB_DIS label removed — GPIO4 now spare (USB charging removed in 2S redesign)
   (global_label "SOLAR_DET" (shape input) (at 220.00 360.00 0) (fields_autoplaced)
     (effects (font (size 1.27 1.27)) (justify left))
@@
     (property "Intersheets" "" (at 0 0 0) (effects (font (size 1.27 1.27)) (hide yes)))
   )
-  (global_label "MAX_ALRT" (shape input) (at 340.00 360.00 0) (fields_autoplaced)
-    (effects (font (size 1.27 1.27)) (justify left))
-    (property "Intersheets" "" (at 0 0 0) (effects (font (size 1.27 1.27)) (hide yes)))
-  )
+  ;; MAX_ALRT label removed — MAX17048 deleted in 2S redesign; GPIO14 now spare
   (global_label "LOOP_TERM_CH1" (shape passive) (at 415.00 175.00 0) (fields_autoplaced)
     (effects (font (size 1.27 1.27)) (justify left))
@@
     (property "Reference" "U7" (at 100.00 41.19 0)
       (effects (font (size 1.27 1.27))))
-    (property "Value" "CN3791" (at 100.00 48.81 0)
+    (property "Value" "CN3722" (at 100.00 48.81 0)
       (effects (font (size 1.27 1.27))))
     (property "Footprint" "" (at 0 0 0)
@@
     (property "Reference" "J1" (at 220.00 76.19 0)
       (effects (font (size 1.27 1.27))))
-    (property "Value" "LiPo" (at 220.00 83.81 0)
+    (property "Value" "LiPo_2S_JST-PH2" (at 220.00 83.81 0)
       (effects (font (size 1.27 1.27))))
     (property "Footprint" "" (at 0 0 0)
@@
     (property "Reference" "U1" (at 340.00 76.19 0)
       (effects (font (size 1.27 1.27))))
-    (property "Value" "TPS7A0533" (at 340.00 83.81 0)
+    (property "Value" "AP63205WU" (at 340.00 83.81 0)
       (effects (font (size 1.27 1.27))))
     (property "Footprint" "" (at 0 0 0)
@@
     (property "Reference" "R7" (at 490.00 86.19 0)
       (effects (font (size 1.27 1.27))))
-    (property "Value" "100k" (at 490.00 93.81 0)
+    (property "Value" "330k" (at 490.00 93.81 0)
       (effects (font (size 1.27 1.27))))
     (property "Footprint" "" (at 0 0 0)
@@
     (property "Reference" "U8" (at 40.00 296.19 0)
       (effects (font (size 1.27 1.27))))
-    (property "Value" "TPS61023" (at 40.00 303.81 0)
+    (property "Value" "MT3608B" (at 40.00 303.81 0)
       (effects (font (size 1.27 1.27))))
     (property "Footprint" "" (at 0 0 0)
@@
     (property "Reference" "R23" (at 120.00 311.19 0)
       (effects (font (size 1.27 1.27))))
-    (property "Value" "1.1M" (at 120.00 318.81 0)
+    (property "Value" "1.9M" (at 120.00 318.81 0)
       (effects (font (size 1.27 1.27))))
     (property "Footprint" "" (at 0 0 0)
@@
     (property "Reference" "R24" (at 160.00 311.19 0)
       (effects (font (size 1.27 1.27))))
-    (property "Value" "47k" (at 160.00 318.81 0)
+    (property "Value" "100k" (at 160.00 318.81 0)
       (effects (font (size 1.27 1.27))))
     (property "Footprint" "" (at 0 0 0)
@@
     (property "Reference" "D8" (at 80.00 311.19 0)
       (effects (font (size 1.27 1.27))))
-    (property "Value" "SMAJ7.0A" (at 80.00 318.81 0)
+    (property "Value" "SMAJ28CA" (at 80.00 318.81 0)
       (effects (font (size 1.27 1.27))))
     (property "Footprint" "" (at 0 0 0)
@@
     (property "Reference" "TP11" (at 350.00 366.19 0)
       (effects (font (size 1.27 1.27))))
-    (property "Value" "VBAT_RAW" (at 350.00 373.81 0)
+    (property "Value" "VBAT_RAW_2S" (at 350.00 373.81 0)
       (effects (font (size 1.27 1.27))))
     (property "Footprint" "" (at 0 0 0)
@@
     (property "Reference" "TP13" (at 380.00 366.19 0)
       (effects (font (size 1.27 1.27))))
-    (property "Value" "MAX_ALRT" (at 380.00 373.81 0)
+    (property "Value" "REMOVED_MAX_ALRT" (at 380.00 373.81 0)
       (effects (font (size 1.27 1.27))))
     (property "Footprint" "" (at 0 0 0)
@@
     (property "Reference" "TP14" (at 395.00 366.19 0)
       (effects (font (size 1.27 1.27))))
-    (property "Value" "/CHRG_SOLAR" (at 395.00 373.81 0)
-      (effects (font (size 1.27 1.27))))
-    (property "Footprint" "" (at 0 0 0)
+    (property "Value" "REMOVED_CHRG_SOLAR" (at 395.00 373.81 0)
+      (effects (font (size 1.27 1.27))))
+    (property "Footprint" "" (at 0 0 0)
