File: hardware/pcb/welld.kicad_sch (KiCad schematic)
At the start: 122 parts, among them J1 LiPo_2S_JST-PH2, J10 PROG_6pin, J12 SolarPanel, J2 USB-C, J3 U.FL_Antenna, J4 4-20mA_CH1, J5 4-20mA_CH2, J6 DS18B20, J7 Spare, J8 I2C_4pin, J9 GPIO_8pin, Q1 BSS123, Q2 BSS123, Q3 BSS84, SW1 RESET, SW2 BOOT, U1 AP63205WU, U10 MAX17048, U2 TP4056, U3 S-8261AAYFT, U4 FS8205A, U5 USBLC6-2SC6, U6 ESP32-C6-MINI, U7 CN3722, U8 MT3608B, U9 ADS1115

Commit message: feat(pcb): generate KiCad 10-compatible schematic with working GUI symbol rendering
Rewrote generate_kicad.py to produce lib_symbols entries with the full
"Library:Name" prefix required by KiCad 10's GUI (e.g. "Device:R",
"welld:AP63205WU", "power:VBAT"). kicad-cli tolerates bare names but
the GUI showed "??" for every symbol without the prefix.

Also adds: stdlib symbol embedding (_extract_sym + _STDLIB_NEEDED),
custom VBAT power symbol, welld.kicad_sym library file, project-level
sym-lib-table with absolute paths, and kicad-cli post-upgrade step.

Removes stale jlcpcb_bom.csv / jlcpcb_cpl.csv (superseded by welld_bom.csv).

Co-Authored-By: Claude Sonnet 4.6 <noreply@anthropic.com>
Parts:
- removed C1, C2: 10uF, symbol Device:C
- removed C16: 4.7uF, symbol Device:C
- removed C25, C26: 100nF, symbol Device:C
- removed D10, D9: SMAJ3.3CA, symbol Device:D_TVS_Bidirectional
- removed D2, D3: LED DNF, symbol Device:LED
- removed F1: PTC 1A, symbol Device:Polyfuse
- removed J2: USB-C, symbol welld:USB_C_Power
- removed Q1, Q2: BSS123, symbol Device:Q_NMOS_GSD
- removed Q3: BSS84, symbol Device:Q_PMOS_GSD
- removed R1: 2.0k, symbol Device:R
- removed R15, R16: 5.1k, symbol Device:R
- removed R17, R18: 1k DNF, symbol Device:R
- removed R25, R27, R29: 4.7k, symbol Device:R
- removed R30: 10k, symbol Device:R
- removed SW1: RESET, symbol Device:SW_Push
- removed SW2: BOOT, symbol Device:SW_Push
- removed TP13: REMOVED_MAX_ALRT, symbol welld:TestPoint_Pad
- removed U1: AP63205WU, symbol welld:TPS7A0533
- removed U10: MAX17048, symbol welld:MAX17048
- removed U2: TP4056, symbol welld:TP4056
- removed U3: S-8261AAYFT, symbol welld:S8261A
- removed U4: FS8205A, symbol welld:FS8205A
- removed U5: USBLC6-2SC6, symbol welld:USBLC6_2SC6
- removed U7: CN3722, symbol welld:CN3791
- removed U8: MT3608B, symbol welld:TPS61023
- added C27: 4.7uF 10V, Capacitor_SMD:C_0805_2012Metric, symbol Device:C
- added C28, C_BUCK: 10uF 10V, Capacitor_SMD:C_0805_2012Metric, symbol Device:C
- added C29: 10uF 16V, Capacitor_SMD:C_0805_2012Metric, symbol Device:C
- added C_BST: 100nF 16V, Capacitor_SMD:C_0402_1005Metric, symbol Device:C
- added D10, D9: SMAJ3.3CA, Diode_SMD:D_SMA, symbol Device:D_TVS
- added D12: PRTR5V0U2X, Package_TO_SOT_SMD:SOT-363_SC-70-6, symbol welld:PRTR5V0U2X
- added D13: SMAJ10CA, Diode_SMD:D_SMA, symbol Device:D_TVS
- added D14: SMAJ28CA, Diode_SMD:D_SMA, symbol Device:D_TVS
- added F2: MF-MSMF110/16X, Fuse:Fuse_1206_3216Metric, symbol Device:Polyfuse
- added J13: USB4135-GF-A, welld:USB_C_GCT_USB4135-GF-A, symbol welld:USB_C_Power
- added L2: 4.7uH, Inductor_SMD:L_2520_6332Metric, symbol Device:L
- added Q2: BSS123, Package_TO_SOT_SMD:SOT-23, symbol Device:Q_NMOS
- added R33: 604k 1%, Resistor_SMD:R_0402_1005Metric, symbol Device:R
- added R34: 100k 1%, Resistor_SMD:R_0402_1005Metric, symbol Device:R
- added R35: 1k2 1%, Resistor_SMD:R_0402_1005Metric, symbol Device:R
- added R36: 100k, Resistor_SMD:R_0402_1005Metric, symbol Device:R
- added R37, R38: 4k7, Resistor_SMD:R_0402_1005Metric, symbol Device:R
- added R_CC1, R_CC2: 5k1, Resistor_SMD:R_0402_1005Metric, symbol Device:R
- added SW1: RESET, Button_Switch_SMD:SW_SPST_PTS636, symbol Switch:SW_Push
- added SW2: BOOT, Button_Switch_SMD:SW_SPST_PTS636, symbol Switch:SW_Push
- added TP15: /CHRG_USB, TestPoint:TestPoint_Pad_1.0x1.0mm, symbol welld:TestPoint_Pad
- added U1: AP63205WU, Package_TO_SOT_SMD:SOT-23-6, symbol welld:AP63205WU
- added U11: USBLC6-2SC6, Package_TO_SOT_SMD:SOT-23-6, symbol welld:USBLC6_2SC6
- added U12: TP5100, Package_SO:SOIC-8_3.9x4.9mm_P1.27mm, symbol welld:TP5100
- added U7: CN3722, Package_SO:SOIC-8_3.9x4.9mm_P1.27mm, symbol welld:CN3722
- added U8: MT3608B, Package_TO_SOT_SMD:SOT-23-6, symbol welld:MT3608B
- C10: value 1uF -> 1uF 16V; footprint (none) -> Capacitor_SMD:C_0402_1005Metric
- C11, C12, C13, C14a, C14b, C14c, C14d, C21, C23, C24, C3, C5, C7, C8, C_SH1, C_SH2: footprint (none) -> Capacitor_SMD:C_0402_1005Metric
- C15, C4, C6: value 10uF -> 10uF 10V; footprint (none) -> Capacitor_SMD:C_0805_2012Metric
- C17: value 10uF -> 10uF 25V; footprint (none) -> Capacitor_SMD:C_0805_2012Metric
- C18, C19, C22: value 10uF -> 10uF 16V; footprint (none) -> Capacitor_SMD:C_0805_2012Metric
- C20: value 22uF -> 22uF 16V; footprint (none) -> Capacitor_SMD:C_1206_3216Metric
- C9: value 100nF -> 100nF 16V; footprint (none) -> Capacitor_SMD:C_0402_1005Metric
- D1: footprint (none) -> Package_TO_SOT_SMD:SOT-363_SC-70-6; LCSC (none) -> C2687116
- D11: footprint (none) -> Diode_SMD:D_SMA; LCSC (none) -> C8057
- D4: footprint (none) -> LED_SMD:LED_0603_1608Metric
- D5: footprint (none) -> Package_TO_SOT_SMD:SOT-23; LCSC (none) -> C31417
- D6: value MBRS140 -> MBRS140T3G; footprint (none) -> Diode_SMD:D_SOD-123
- D7: value LED DNF -> Solar_LED_DNF; footprint (none) -> LED_SMD:LED_0603_1608Metric
- D8: footprint (none) -> Diode_SMD:D_SMA
- FB1: footprint (none) -> Inductor_SMD:L_0402_1005Metric; LCSC (none) -> C76537
- J1: value LiPo_2S_JST-PH2 -> B2B-PH-K-S; footprint (none) -> Connector_JST:JST_PH_B2B-PH-K_1x02_P2.00mm_Vertical; LCSC (none) -> C457925
- J10: footprint (none) -> Connector_PinHeader_1.27mm:PinHeader_1x06_P1.27mm_Vertical
- J12: value SolarPanel -> MC 1.5/2-G-3.5; footprint (none) -> TerminalBlock_Phoenix:TerminalBlock_Phoenix_MC-1.5_2pin_3.5mm
- J3: value U.FL_Antenna -> U.FL; footprint (none) -> Connector_Coaxial:U.FL_Hirose_U.FL-R-SMT-1_Vertical
- J4, J5, J6, J7: footprint (none) -> TerminalBlock_Phoenix:TerminalBlock_Phoenix_MC-1.5_3pin_3.5mm
- J8: footprint (none) -> Connector_PinHeader_2.54mm:PinHeader_1x04_P2.54mm_Vertical
- J9: footprint (none) -> Connector_PinHeader_2.54mm:PinHeader_1x08_P2.54mm_Vertical
- L1: footprint (none) -> Inductor_SMD:L_4x4mm; LCSC (none) -> C376098
- R10, R26, R6, R9: value 4.7k -> 4k7; footprint (none) -> Resistor_SMD:R_0402_1005Metric
- R11, R12, R13, R14, R22, R28, R3, R31, R32, R5: footprint (none) -> Resistor_SMD:R_0402_1005Metric
- R19: value 2k -> 2k0 1%; footprint (none) -> Resistor_SMD:R_0402_1005Metric
- R2, R4: footprint (none) -> Resistor_SMD:R_0805_2012Metric
- R20: value 36k -> 36k 1%; footprint (none) -> Resistor_SMD:R_0402_1005Metric
- R21: value 10k -> 10k 1%; footprint (none) -> Resistor_SMD:R_0402_1005Metric
- R23: value 1.9M -> 1.91M 1%; footprint (none) -> Resistor_SMD:R_0402_1005Metric
- R24, R8: value 100k -> 100k 1%; footprint (none) -> Resistor_SMD:R_0402_1005Metric
- R7: value 330k -> 330k 1%; footprint (none) -> Resistor_SMD:R_0402_1005Metric
- SJ1, SJ2, SJ3, SJ4, SJ5: footprint (none) -> Jumper:SolderJumper_2_Open
- TP1, TP10, TP12, TP2, TP3, TP4, TP5, TP6, TP7, TP8, TP9: footprint (none) -> TestPoint:TestPoint_Pad_1.0x1.0mm
- TP11: value VBAT_RAW_2S -> VBAT_RAW; footprint (none) -> TestPoint:TestPoint_Pad_1.0x1.0mm
- TP14: value REMOVED_CHRG_SOLAR -> /CHRG_SOLAR; footprint (none) -> TestPoint:TestPoint_Pad_1.0x1.0mm
- U6: value ESP32-C6-MINI -> ESP32-C6-MINI-1U-H4; footprint (none) -> welld:ESP32_C6_MINI_1U
- U9: value ADS1115 -> ADS1115IDGST; footprint (none) -> Package_SO:MSOP-10_3x3mm_P0.5mm; LCSC (none) -> C37593

Commit message: hw(pcb): full placement pass, XT30 connector, SMA antenna, BOM cleanup
Component placement:
- All 116 components placed inside 80×55 mm board outline
- pcbway_cpl.csv fully rewritten with correct board-relative coordinates

Battery connector (J1):
- Changed from JST PH 2.0mm to AMASS XT30PW-F right-angle THT (LCSC C601498)
- Pad drill corrected 1.5 mm → 1.8 mm for IPC-2221 wave-solder clearance

Antenna (J3 + W1):
- J3: Amphenol 132289 SMD edge-launch SMA on bottom board edge
- W1: Taoglas CAB.100.07.0050B ~50 mm U.FL-to-SMA pigtail (hand-attached post-reflow)
- RF_ANT net assigned to J3 signal pad

Inductor L2:
- Footprint corrected from L_2512_6332Metric to L_Vishay_IFSC-1515AH_4x4x1.8mm
- Now matches MPN CDRH4D22NP-4R7NC body; shares footprint, reel, and LCSC C376098 with L1

VLOOP output caps (C20, C22):
- Voltage rating upgraded 16 V → 25 V (2.1× margin on 12 V rail; proper DC-bias headroom)
- Footprints unchanged (1206 / 0805)

BOM cleanup:
- J8, J9: marked DNF (expansion headers not populated in production)
- J4–J7, J12, J10: Package updated to THT; PCBWay wave-solders

Case:
- XT30PW-F left-wall cutout added: 14×12 mm slot at Y=17–31 mm, Z=19.3–31.3 mm
- SMA bottom-wall cutout (10.5 mm ⌀ at X=42.5 mm) confirmed present

Co-Authored-By: Claude Sonnet 4.6 <noreply@anthropic.com>
Parts:
- removed C10: 1uF 16V, Capacitor_SMD:C_0402_1005Metric, symbol Device:C
- removed C11, C13, C14a, C14b, C14c, C14d, C21, C23, C7, C8: 100nF, Capacitor_SMD:C_0402_1005Metric, symbol Device:C
- removed C12, C24, C3, C5: 1uF, Capacitor_SMD:C_0402_1005Metric, symbol Device:C
- removed C15, C28, C4, C6, C_BUCK: 10uF 10V, Capacitor_SMD:C_0805_2012Metric, symbol Device:C
- removed C17: 10uF 25V, Capacitor_SMD:C_0805_2012Metric, symbol Device:C
- removed C18, C19, C22, C29: 10uF 16V, Capacitor_SMD:C_0805_2012Metric, symbol Device:C
- removed C20: 22uF 16V, Capacitor_SMD:C_1206_3216Metric, symbol Device:C
- removed C27: 4.7uF 10V, Capacitor_SMD:C_0805_2012Metric, symbol Device:C
- removed C9, C_BST: 100nF 16V, Capacitor_SMD:C_0402_1005Metric, symbol Device:C
- removed C_SH1, C_SH2: 10nF, Capacitor_SMD:C_0402_1005Metric, symbol Device:C
- removed D1, D12: PRTR5V0U2X, Package_TO_SOT_SMD:SOT-363_SC-70-6, symbol welld:PRTR5V0U2X
- removed D10, D9: SMAJ3.3CA, Diode_SMD:D_SMA, symbol Device:D_TVS
- removed D11: SMAJ13A, Diode_SMD:D_SMA, symbol Device:D_TVS
- removed D13: SMAJ10CA, Diode_SMD:D_SMA, symbol Device:D_TVS
- removed D14, D8: SMAJ28CA, Diode_SMD:D_SMA, symbol Device:D_TVS
- removed D4: Status_LED, LED_SMD:LED_0603_1608Metric, symbol Device:LED
- removed D5: AO3407, Package_TO_SOT_SMD:SOT-23, symbol welld:AO3407
- removed D6: MBRS140T3G, Diode_SMD:D_SOD-123, symbol Device:D_Schottky
- removed D7: Solar_LED_DNF, LED_SMD:LED_0603_1608Metric, symbol Device:LED
- removed F2: MF-MSMF110/16X, Fuse:Fuse_1206_3216Metric, symbol Device:Polyfuse
- removed FB1: BLM18KG601SN1D, Inductor_SMD:L_0402_1005Metric, symbol Device:L
- removed J1: B2B-PH-K-S, Connector_JST:JST_PH_B2B-PH-K_1x02_P2.00mm_Vertical, symbol Connector:Conn_01x02_Pin
- removed J10: PROG_6pin, Connector_PinHeader_1.27mm:PinHeader_1x06_P1.27mm_Vertical, symbol Connector:Conn_01x06_Pin
- removed J12: MC 1.5/2-G-3.5, TerminalBlock_Phoenix:TerminalBlock_Phoenix_MC-1.5_2pin_3.5mm, symbol Connector:Conn_01x02_Pin
- removed J13: USB4135-GF-A, welld:USB_C_GCT_USB4135-GF-A, symbol welld:USB_C_Power
- removed J3: U.FL, Connector_Coaxial:U.FL_Hirose_U.FL-R-SMT-1_Vertical, symbol welld:U_FL_Antenna
- removed J4: 4-20mA_CH1, TerminalBlock_Phoenix:TerminalBlock_Phoenix_MC-1.5_3pin_3.5mm, symbol Connector:Conn_01x03_Pin
- removed J5: 4-20mA_CH2, TerminalBlock_Phoenix:TerminalBlock_Phoenix_MC-1.5_3pin_3.5mm, symbol Connector:Conn_01x03_Pin
- removed J6: DS18B20, TerminalBlock_Phoenix:TerminalBlock_Phoenix_MC-1.5_3pin_3.5mm, symbol Connector:Conn_01x03_Pin
- removed J7: Spare, TerminalBlock_Phoenix:TerminalBlock_Phoenix_MC-1.5_3pin_3.5mm, symbol Connector:Conn_01x03_Pin
- removed J8: I2C_4pin, Connector_PinHeader_2.54mm:PinHeader_1x04_P2.54mm_Vertical, symbol Connector:Conn_01x04_Pin
- removed J9: GPIO_8pin, Connector_PinHeader_2.54mm:PinHeader_1x08_P2.54mm_Vertical, symbol Connector:Conn_01x08_Pin
- removed L1: 4.7uH, Inductor_SMD:L_4x4mm, symbol Device:L
- removed L2: 4.7uH, Inductor_SMD:L_2520_6332Metric, symbol Device:L
- removed Q2: BSS123, Package_TO_SOT_SMD:SOT-23, symbol Device:Q_NMOS
- removed R10, R26, R37, R38, R6, R9: 4k7, Resistor_SMD:R_0402_1005Metric, symbol Device:R
- removed R11, R12, R13, R31: 10k, Resistor_SMD:R_0402_1005Metric, symbol Device:R
- removed R14: 1k, Resistor_SMD:R_0402_1005Metric, symbol Device:R
- removed R19: 2k0 1%, Resistor_SMD:R_0402_1005Metric, symbol Device:R
- removed R2, R4: 100R 0.1%, Resistor_SMD:R_0805_2012Metric, symbol Device:R
- removed R20: 36k 1%, Resistor_SMD:R_0402_1005Metric, symbol Device:R
- removed R21: 10k 1%, Resistor_SMD:R_0402_1005Metric, symbol Device:R
- removed R22: 1k DNF, Resistor_SMD:R_0402_1005Metric, symbol Device:R
- removed R23: 1.91M 1%, Resistor_SMD:R_0402_1005Metric, symbol Device:R
- removed R24, R34, R8: 100k 1%, Resistor_SMD:R_0402_1005Metric, symbol Device:R
- removed R28, R3, R5: 100R, Resistor_SMD:R_0402_1005Metric, symbol Device:R
- removed R32: 33R DNF, Resistor_SMD:R_0402_1005Metric, symbol Device:R
- removed R33: 604k 1%, Resistor_SMD:R_0402_1005Metric, symbol Device:R
- removed R35: 1k2 1%, Resistor_SMD:R_0402_1005Metric, symbol Device:R
- removed R36: 100k, Resistor_SMD:R_0402_1005Metric, symbol Device:R
- removed R7: 330k 1%, Resistor_SMD:R_0402_1005Metric, symbol Device:R
- removed R_CC1, R_CC2: 5k1, Resistor_SMD:R_0402_1005Metric, symbol Device:R
- removed SJ1: VBOOST_EN DNF, Jumper:SolderJumper_2_Open, symbol Jumper:SolderJumper_2_Open
- removed SJ2: VLOOP_BUS, Jumper:SolderJumper_2_Open, symbol Jumper:SolderJumper_2_Open
- removed SJ3: LED_DIS, Jumper:SolderJumper_2_Open, symbol Jumper:SolderJumper_2_Open
- removed SJ4: UART_TX DNF, Jumper:SolderJumper_2_Open, symbol Jumper:SolderJumper_2_Open
- removed SJ5: UART_RX DNF, Jumper:SolderJumper_2_Open, symbol Jumper:SolderJumper_2_Open
- removed SW1: RESET, Button_Switch_SMD:SW_SPST_PTS636, symbol Switch:SW_Push
- removed SW2: BOOT, Button_Switch_SMD:SW_SPST_PTS636, symbol Switch:SW_Push
- removed TP1: VBAT, TestPoint:TestPoint_Pad_1.0x1.0mm, symbol welld:TestPoint_Pad
- removed TP10: VSOLAR_IN, TestPoint:TestPoint_Pad_1.0x1.0mm, symbol welld:TestPoint_Pad
- removed TP11: VBAT_RAW, TestPoint:TestPoint_Pad_1.0x1.0mm, symbol welld:TestPoint_Pad
- removed TP12: ADS_DRDY, TestPoint:TestPoint_Pad_1.0x1.0mm, symbol welld:TestPoint_Pad
- removed TP14: /CHRG_SOLAR, TestPoint:TestPoint_Pad_1.0x1.0mm, symbol welld:TestPoint_Pad
- removed TP15: /CHRG_USB, TestPoint:TestPoint_Pad_1.0x1.0mm, symbol welld:TestPoint_Pad
- removed TP2: VLOOP, TestPoint:TestPoint_Pad_1.0x1.0mm, symbol welld:TestPoint_Pad
- removed TP3: +3V3, TestPoint:TestPoint_Pad_1.0x1.0mm, symbol welld:TestPoint_Pad
- removed TP4: GND, TestPoint:TestPoint_Pad_1.0x1.0mm, symbol welld:TestPoint_Pad
- removed TP5: LOOP_TERM_CH1, TestPoint:TestPoint_Pad_1.0x1.0mm, symbol welld:TestPoint_Pad
- removed TP6: LOOP_TERM_CH2, TestPoint:TestPoint_Pad_1.0x1.0mm, symbol welld:TestPoint_Pad
- removed TP7: 1WIRE, TestPoint:TestPoint_Pad_1.0x1.0mm, symbol welld:TestPoint_Pad
- removed TP8: I2C_SDA, TestPoint:TestPoint_Pad_1.0x1.0mm, symbol welld:TestPoint_Pad
- removed TP9: I2C_SCL, TestPoint:TestPoint_Pad_1.0x1.0mm, symbol welld:TestPoint_Pad
- removed U1: AP63205WU, Package_TO_SOT_SMD:SOT-23-6, symbol welld:AP63205WU
- removed U11: USBLC6-2SC6, Package_TO_SOT_SMD:SOT-23-6, symbol welld:USBLC6_2SC6
- removed U12: TP5100, Package_SO:SOIC-8_3.9x4.9mm_P1.27mm, symbol welld:TP5100
- removed U6: ESP32-C6-MINI-1U-H4, welld:ESP32_C6_MINI_1U, symbol welld:ESP32_C6_MINI_1U
- removed U7: CN3722, Package_SO:SOIC-8_3.9x4.9mm_P1.27mm, symbol welld:CN3722
- removed U8: MT3608B, Package_TO_SOT_SMD:SOT-23-6, symbol welld:MT3608B
- removed U9: ADS1115IDGST, Package_SO:MSOP-10_3x3mm_P0.5mm, symbol welld:ADS1115
Connections:
- no-connect marks 1 -> 0
Other:
- added sheet interfaces (interfaces.kicad_sch)
- added sheet mcu (mcu.kicad_sch)
- added sheet power (power.kicad_sch)
- added sheet sensors (sensors.kicad_sch)
