File: hardware/pcb/welld.kicad_pcb (KiCad board)
At the start: 2 copper layers, 80 x 55 mm, 120 parts, among them J1 XT30PW-F, J10 PROG, J12 Solar, J13 USB-C, J3 132289, J4 4-20mA_1, J5 4-20mA_2, J6 DS18B20, J7 Spare, Q2 BSS123, SW1 RESET, SW2 BOOT, U1 AP63205, U11 USBLC6, U12 TP5100, U6 ESP32-C6, U7 CN3722, U8 MT3608B, U9 ADS1115

Commit message: chore(pre-prod): cleanup, align docs with 2S design, fix CI pipeline
Documentation and agent file cleanup:
- Update all stale IC references (MAX17048, TP4056, CN3791, TPS7A0533,
  S-8261AAYFT) to current 2S design (ADS1115, TP5100, CN3722, AP63205)
- Update ESP-IDF version references from v5.3.5 to v6.0.1 everywhere
- Fix J1 connector: JST PH 2.0mm -> AMASS XT30PW-F (LCSC C601498)
- Fix fab house: JLCPCB -> PCBWay throughout hardware/pcb/fab_notes.md
- Update hardware/README.md Option 2 to reflect current 2S1P BOM
- Add DS18B20 GPIO default note to docs/wiring.md (PCB default is GPIO7)
- AGENTS.md and agent definitions aligned to v6.0.1 + 6-job CI
- Remove stale historical IC comments from sensor.h and main.c

CI pipeline:
- Replace all third-party actions (actions/checkout, espressif/esp-idf-ci-action,
  actions/setup-node, actions/upload-artifact) with inline git/docker/shell
  steps to satisfy repo action-ownership policy
- checkout: git init + fetch by SHA
- ESP-IDF builds: docker run espressif/idf:v6.0.1 with mounted workspace
- Node.js: curl nodesource setup_20.x

Hardware (PCB):
- Add XT30PW-M custom KiCad symbol and 3D model to WellD.pretty/
- Add update_placements.py scripted placement tool
- Schematic and layout updates for 2S redesign (interfaces, MCU, power, sensors)
- .gitignore: add __pycache__/, *.pyc, *-erc.json, *-drc.json, .cache/

Co-Authored-By: Claude Sonnet 4.6 <noreply@anthropic.com>
Parts:
- moved J4 8.54 mm to (141.0, 56.5)
- moved J5 8.54 mm to (141.0, 68.5)
- moved J6 8.54 mm to (141.0, 80.5)
- moved TP1 7.00 mm to (75.0, 98.5)
- moved J7 5.00 mm to (141.0, 92.5)
- moved J1 3.00 mm to (70.0, 80.0)
- turned J13 to 180 degrees
Changed lines of the file:
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@@
     )
   )
-  (footprint "Connector_USB:USB_C_Receptacle_GCT_USB4135-GF-A_6P_TopMnt_Horizontal" (layer "F.Cu") (at 70.000 71.500 0.0)
+  (footprint "Connector_USB:USB_C_Receptacle_GCT_USB4135-GF-A_6P_TopMnt_Horizontal" (layer "F.Cu") (at 70.000 71.500 180.0)
     (property "Reference" "J13" (at 0 -1.5 0) (layer "F.SilkS")
       (effects (font (size 0.8 0.8) (thickness 0.12)))
@@
     )
   )
-  (footprint "WellD:XT30PW-F_RightAngle" (layer "F.Cu") (at 67.000 80.000 270.0)
+  (footprint "WellD:XT30PW-F_RightAngle" (layer "F.Cu") (at 70.000 80.000 270.0)
     (property "Reference" "J1" (at 0 -1.5 0) (layer "F.SilkS")
       (effects (font (size 0.8 0.8) (thickness 0.12)))
@@
     )
   )
-  (footprint "TerminalBlock_Phoenix:TerminalBlock_Phoenix_PT-1,5-3-3.5-H_1x03_P3.50mm_Horizontal" (layer "F.Cu") (at 138.000 64.500 180.0)
+  (footprint "TerminalBlock_Phoenix:TerminalBlock_Phoenix_PT-1,5-3-3.5-H_1x03_P3.50mm_Horizontal" (layer "F.Cu") (at 141.000 56.500 180.0)
     (property "Reference" "J4" (at 0 -1.5 0) (layer "F.SilkS")
       (effects (font (size 0.8 0.8) (thickness 0.12)))
@@
     )
   )
-  (footprint "TerminalBlock_Phoenix:TerminalBlock_Phoenix_PT-1,5-3-3.5-H_1x03_P3.50mm_Horizontal" (layer "F.Cu") (at 138.000 76.500 180.0)
+  (footprint "TerminalBlock_Phoenix:TerminalBlock_Phoenix_PT-1,5-3-3.5-H_1x03_P3.50mm_Horizontal" (layer "F.Cu") (at 141.000 68.500 180.0)
     (property "Reference" "J5" (at 0 -1.5 0) (layer "F.SilkS")
       (effects (font (size 0.8 0.8) (thickness 0.12)))
@@
     )
   )
-  (footprint "TerminalBlock_Phoenix:TerminalBlock_Phoenix_PT-1,5-3-3.5-H_1x03_P3.50mm_Horizontal" (layer "F.Cu") (at 138.000 88.500 180.0)
+  (footprint "TerminalBlock_Phoenix:TerminalBlock_Phoenix_PT-1,5-3-3.5-H_1x03_P3.50mm_Horizontal" (layer "F.Cu") (at 141.000 80.500 180.0)
     (property "Reference" "J6" (at 0 -1.5 0) (layer "F.SilkS")
       (effects (font (size 0.8 0.8) (thickness 0.12)))
@@
     )
   )
-  (footprint "TerminalBlock_Phoenix:TerminalBlock_Phoenix_PT-1,5-3-3.5-H_1x03_P3.50mm_Horizontal" (layer "F.Cu") (at 138.000 96.500 180.0)
+  (footprint "TerminalBlock_Phoenix:TerminalBlock_Phoenix_PT-1,5-3-3.5-H_1x03_P3.50mm_Horizontal" (layer "F.Cu") (at 141.000 92.500 180.0)
     (property "Reference" "J7" (at 0 -1.5 0) (layer "F.SilkS")
       (effects (font (size 0.8 0.8) (thickness 0.12)))
@@
     )
   )
-  (footprint "TestPoint:TestPoint_Pad_1.0x1.0mm" (layer "F.Cu") (at 68.000 98.500 0.0)
+  (footprint "TestPoint:TestPoint_Pad_1.0x1.0mm" (layer "F.Cu") (at 75.000 98.500 0.0)
     (property "Reference" "TP1" (at 0 -1.5 0) (layer "F.SilkS")
       (effects (font (size 0.8 0.8) (thickness 0.12)))
