File: hardware/pcb/power.kicad_sch (KiCad schematic)
At the start: 76 parts, among them J12 Solar, J13 USB-C, Q3 AO3407, Q4 AO3400A, Q5 AO3407, Q6 FS8205A, Q7 AO3400A, U1 HT7333-A, U11 USBLC6, U12 TP4056, U13 DW01A, U14 LM393, U7 CN3791, U8 MT3608B

Commit message: hw(pcb): resolve BT1 + HRO USB-C footprints to KiCad-standard parts (fab item #2)
Checked the KiCad standard footprint libraries directly instead of drawing
customs:
- BT1 carrier: use Battery:BatteryHolder_Keystone_1042_1x18650 (KiCad
  standard, exact ~78mm dimensional match: pad 1 = + at -39.33, pad 2 = -
  at +39.33, SMD + 2 alignment posts). Schematic footprint field changed
  from the custom WellD:BH-18650_THT. Populate with a Keystone 1042
  (off-LCSC) or the LCSC MYOUNG BH-18650-B1BA002 (C2988620) if terminals
  match -- no custom draw needed.
- HRO USB-C: Connector_USB:USB_C_Receptacle_HRO_TYPE-C-31-M-12 confirmed
  present in the standard lib (descr matches the krhro.com part; all needed
  A/B/S pads present) -- the 'verify name' warning is cleared.
- GDT land pattern: still open but correctly gated -- GDT1/2 are DNF with
  no chosen MPN, so the pattern is drawn only when a specific part is picked.

Two of three footprint items resolved; the third is deferred by design.
Netlist unchanged: 391 pins / 75 nets / zero mismatches.

Co-Authored-By: Claude Opus 4.8 <noreply@anthropic.com>
Claude-Session: https://claude.ai/code/session_01VtMFY5Q94iYbsNPpLcPJyK
Parts:
- BT1: footprint WellD:BH-18650_THT -> Battery:BatteryHolder_Keystone_1042_1x18650
Changed lines of the file:
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@@
 			)
 		)
-		(property "Footprint" "WellD:BH-18650_THT"
+		(property "Footprint" "Battery:BatteryHolder_Keystone_1042_1x18650"
 			(at 0 0 0)
 			(hide yes)
